Commit message: Update robot to 4-DOF with Panda gripper for ROS 2 Humble
- Remove link_5, link_6, joint_5, joint_6 from URDF
- Add Panda gripper (panda_hand, panda_leftfinger, panda_rightfinger)
- Add gripper joints (panda_finger_joint1, panda_finger_joint2)
- Update ros2_control configuration for gripper
- Update MoveIt configuration files
- Create display_rviz.launch.py for RViz visualization
- Update gazebo.launch.py to load gripper controller
- Update README.md with comprehensive documentation
- Create display.rviz config file

Co-authored-by: PhuocToan180405 <165999379+PhuocToan180405@users.noreply.github.com>

File: six_dof_arm/urdf/six_dof_arm.urdf (robot description, URDF)
Before this commit: robot six_dof_arm, 7 links, 6 joints
Links:
- removed link link_5
- removed link link_6
- added link panda_hand, mass 0.73; collision box size=0.06 0.02 0.08; visual box size=0.06 0.02 0.08
- added link panda_leftfinger, mass 0.1; collision box size=0.01 0.02 0.04; visual box size=0.01 0.02 0.04
- added link panda_rightfinger, mass 0.1; collision box size=0.01 0.02 0.04; visual box size=0.01 0.02 0.04
Joints:
- removed joint joint_5
- removed joint joint_6
- added joint panda_finger_joint1: type prismatic, parent panda_hand, child panda_leftfinger, origin xyz=0 0.02 0.08 rpy=0 0 0, axis 0 1 0, limit lower=0 upper=0.04 effort=20 velocity=0.2
- added joint panda_finger_joint2: type prismatic, parent panda_hand, child panda_rightfinger, origin xyz=0 -0.02 0.08 rpy=0 0 0, axis 0 -1 0, limit lower=0 upper=0.04 effort=20 velocity=0.2
- added joint panda_hand_joint: type fixed, parent link_4, child panda_hand, origin xyz=0.041309 0.030815 0 rpy=-1.5708 -0.5334 -1.5708

File: six_dof_arm_moveit_config/config/six_dof_arm.ros2_control.xacro (robot description, xacro)
@@ -40,17 +40,17 @@
                 <state_interface name="velocity"/>
             </joint>
-            <joint name="joint_5">
+            <joint name="panda_finger_joint1">
                 <command_interface name="position"/>
                 <command_interface name="velocity"/>
                 <state_interface name="position">
-                  <param name="initial_value">${initial_positions['joint_5']}</param>
+                  <param name="initial_value">0.04</param>
                 </state_interface>
                 <state_interface name="velocity"/>
             </joint>
-            <joint name="joint_6">
+            <joint name="panda_finger_joint2">
                 <command_interface name="position"/>
                 <command_interface name="velocity"/>
                 <state_interface name="position">
-                  <param name="initial_value">${initial_positions['joint_6']}</param>
+                  <param name="initial_value">0.04</param>
                 </state_interface>
                 <state_interface name="velocity"/>
